File: esp-test.kicad_sch (KiCad schematic)
At the start: 9 parts, among them U1 ESP32-S3-WROOM-1

Commit message: work
Parts:
- removed 5.1 kΩ: R_US, symbol Device:R_US (x2)
- added 2kΩ, 470Ω: R_US, symbol Device:R_US
- added 5.1 kΩ: R_Small, symbol Device:R_Small
- added 5.1 kΩ1: R_Small, symbol Device:R_Small
- added C1, C2, C3, C4: 4.7 µF, symbol Device:C_Small_US
- added D1: Charge Indicator, symbol Device:LED
- added J1: AudioPlug3, symbol Connector_Audio:AudioPlug3
- added SW1: SW_SPST, symbol Switch:SW_SPST
- added U2: AP2112K-3.3, Package_TO_SOT_SMD:SOT-23-5, symbol Regulator_Linear:AP2112K-3.3
- added U3: PCM5102A, Package_SO:TSSOP-20_4.4x6.5mm_P0.65mm, symbol Audio:PCM5102A
- added U4: TPA6132A2RTE, Package_DFN_QFN:WQFN-16-1EP_3x3mm_P0.5mm_EP1.6x1.6mm_ThermalVias, symbol Amplifier_Audio:TPA6132A2RTE
Connections:
- net GND: now also U1.1 (GND), U1.40 (GND), U1.41 (GND), 2kΩ.2, 5.1 kΩ.2, 5.1 kΩ1.2, C1.1, C2.1, C3.1, C4.1, U2.2 (GND)
- net at USB-C Connector.A5 (CC1): now also 5.1 kΩ.1
- net at USB-C Connector.A6 (D+), USB-C Connector.B6 (D+): now also USBLC6-2SC6.3 (I/O2); no longer USBLC6-2SC6.1 (I/O1)
- net at USB-C Connector.A7 (D-), USB-C Connector.B7 (D-): now also USBLC6-2SC6.1 (I/O1); no longer USBLC6-2SC6.3 (I/O2)
- net at USB-C Connector.B5 (CC2): now also 5.1 kΩ1.1
- net at F1.2, MCP73831.4 (V_{DD}), USBLC6-2SC6.5 (VBUS): now also C1.2, D1.2 (A)
- net at JST PH 2.0 2-pin.1 (Pin_1), MCP73831.3 (V_{BAT}): now also C2.2, C3.2, SW1.1 (A), U2.1 (VIN)
- net at USBLC6-2SC6.4 (I/O2): now also U1.14 (USB_D+); no longer U1.13 (USB_D-)
- net at USBLC6-2SC6.6 (I/O1): now also U1.13 (USB_D-); no longer U1.14 (USB_D+)
- net at MCP73831.1 (STAT): now also 470Ω.1
- net at MCP73831.5 (PROG): now also 2kΩ.1
- net at U1.2 (3V3): now also C4.2, U2.5 (VOUT)
- new net: SW1.2 (B), U2.3 (EN)
- new net: 470Ω.2, D1.1 (K)
Other:
- moved on the sheet: BT1, JST PH 2.0 2-pin, MCP73831, USB-C Connector, USBLC6-2SC6

Commit message: work
Parts:
- renumbered U4 to Amplifier, U3 to DAC, SW1 to PowerSwitch
Connections:
- net at DAC.13 (BCK): now also U1.7 (IO7)
- net at DAC.14 (DIN): now also U1.6 (IO6)
- net at DAC.15 (LRCK): now also U1.5 (IO5)
- no-connect marks 2 -> 3
Other:
- moved on the sheet: Amplifier, DAC, J1
Changed lines of the file:
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@@
 		(at 57.15 127)
 	)
+	(no_connect
+		(at 180.34 129.54)
+	)
 	(wire
 		(pts
@@
 	(wire
 		(pts
+			(xy 160.02 121.92) (xy 180.34 121.92)
+		)
+		(stroke
+			(width 0)
+			(type default)
+		)
+	)
+	(wire
+		(pts
 			(xy 113.03 74.93) (xy 116.84 74.93)
 		)
@@
 	(wire
 		(pts
+			(xy 160.02 124.46) (xy 180.34 124.46)
+		)
+		(stroke
+			(width 0)
+			(type default)
+		)
+	)
+	(wire
+		(pts
 			(xy 107.95 88.9) (xy 107.95 72.39)
 		)
@@
 		(pts
 			(xy 60.96 83.82) (xy 76.2 83.82)
+		)
+		(stroke
+			(width 0)
+			(type default)
+		)
+	)
+	(wire
+		(pts
+			(xy 160.02 127) (xy 180.34 127)
 		)
 		(stroke
@@
 	(symbol
 		(lib_id "Amplifier_Audio:TPA6132A2RTE")
-		(at 200.66 140.97 0)
+		(at 261.62 113.03 0)
 		(unit 1)
 		(exclude_from_sim no)
@@
 		(dnp no)
 		(fields_autoplaced yes)
-		(property "Reference" "U4"
-			(at 202.8033 123.19 0)
+		(property "Reference" "Amplifier"
+			(at 263.7633 95.25 0)
 			(effects
 				(font
@@
 		)
 		(property "Value" "TPA6132A2RTE"
-			(at 202.8033 125.73 0)
+			(at 263.7633 97.79 0)
 			(effects
 				(font
@@
 		)
 		(property "Footprint" "Package_DFN_QFN:WQFN-16-1EP_3x3mm_P0.5mm_EP1.6x1.6mm_ThermalVias"
-			(at 203.2 154.94 0)
+			(at 264.16 127 0)
 			(effects
 				(font
@@
 		)
 		(property "Datasheet" "https://www.ti.com/lit/ds/symlink/tpa6132a2.pdf"
-			(at 193.04 127 0)
+			(at 254 99.06 0)
 			(effects
 				(font
@@
 		)
 		(property "Description" "25mW, Stereo, DirectPath Audio Amplifier, WQFN-16"
-			(at 200.66 140.97 0)
+			(at 261.62 113.03 0)
 			(effects
 				(font
@@
 			(project ""
 				(path "/555abb5d-59e2-4269-9cc6-b55b0714b43e"
-					(reference "U4")
+					(reference "Amplifier")
 					(unit 1)
 				)
@@
 		(on_board yes)
 		(dnp no)
-		(fields_autoplaced yes)
-		(property "Reference" "SW1"
-			(at 118.11 92.71 0)
-			(effects
-				(font
-					(size 1.27 1.27)
+		(property "Reference" "PowerSwitch"
+			(at 118.11 96.012 0)
+			(effects
+				(font
+					(size 0.762 0.762)
 				)
 			)
@@
 					(size 1.27 1.27)
 				)
+				(hide yes)
 			)
 		)
@@
 			(project ""
 				(path "/555abb5d-59e2-4269-9cc6-b55b0714b43e"
-					(reference "SW1")
+					(reference "PowerSwitch")
 					(unit 1)
 				)
@@
 	(symbol
 		(lib_id "Connector_Audio:AudioPlug3")
-		(at 176.53 59.69 0)
+		(at 260.35 83.82 0)
 		(unit 1)
 		(exclude_from_sim no)
@@
 		(fields_autoplaced yes)
 		(property "Reference" "J1"
-			(at 176.53 49.53 0)
+			(at 260.35 73.66 0)
 			(effects
 				(font
@@
 		)
 		(property "Value" "AudioPlug3"
-			(at 176.53 52.07 0)
+			(at 260.35 76.2 0)
 			(effects
 				(font
@@
 		)
 		(property "Footprint" ""
-			(at 179.07 60.96 0)
+			(at 262.89 85.09 0)
 			(effects
 				(font
@@
 		)
 		(property "Datasheet" "~"
-			(at 179.07 60.96 0)
+			(at 262.89 85.09 0)
 			(effects
 				(font
@@
 		)
 		(property "Description" "Audio Jack, 3 Poles (Stereo / TRS)"
-			(at 176.53 59.69 0)
+			(at 260.35 83.82 0)
 			(effects
 				(font
@@
 	(symbol
 		(lib_id "Audio:PCM5102A")
-		(at 200.66 92.71 0)
+		(at 193.04 132.08 0)
 		(unit 1)
 		(exclude_from_sim no)
@@
 		(dnp no)
 		(fields_autoplaced yes)
-		(property "Reference" "U3"
-			(at 205.3433 74.93 0)
+		(property "Reference" "DAC"
+			(at 197.7233 114.3 0)
 			(effects
 				(font
@@
 		)
 		(property "Value" "PCM5102A"
-			(at 205.3433 77.47 0)
+			(at 197.7233 116.84 0)
 			(effects
 				(font
@@
 		)
 		(property "Footprint" "Package_SO:TSSOP-20_4.4x6.5mm_P0.65mm"
-			(at 226.06 109.22 0)
+			(at 218.44 148.59 0)
 			(effects
 				(font
@@
 		)
 		(property "Datasheet" "https://www.ti.com/lit/ds/symlink/pcm5102a.pdf"
-			(at 200.66 92.71 0)
+			(at 193.04 132.08 0)
 			(effects
 				(font
@@
 		)
 		(property "Description" "2.1 VRMS, 112dB Audio Stereo DAC with PLL and 32-bit, 384kHz PCM Interface, TSSOP-20"
-			(at 200.66 92.71 0)
+			(at 193.04 132.08 0)
 			(effects
 				(font
@@
 			(project ""
 				(path "/555abb5d-59e2-4269-9cc6-b55b0714b43e"
-					(reference "U3")
-					(unit 1)
-				)
+					(reference "DAC")
+					(unit 1)
+				)

Commit message: work
Parts:
- added 470Ω, 470Ω1: R_US, symbol Device:R_US
- added C10, C14, C6, C8: 0.1 µF, symbol Device:C_Small
- added C11, C13, C5, C9: 10 µF, symbol Device:C_Small_US
- added C12, C17, C18, C7: 2.2 µF, symbol Device:C_Small
- added C15, C16: 1 µF, symbol Device:C_Small
- added FB1: FerriteBead, symbol Device:FerriteBead
Connections:
- net GND: now also DAC.10 (DEMP), DAC.11 (FLT), DAC.16 (FMT), DAC.19 (DGND), DAC.20 (DVDD), C13.1, C13.2, C14.1, C14.2, C5.2, C6.2
- net at C4.2, U1.2 (3V3), U2.5 (VOUT): now also FB1.1
- net GNDA: now reaches Amplifier.1 (INL-)
- net GNDA: now also Amplifier.4 (INR-), DAC.3 (CPGND), DAC.9 (AGND), 470Ω.2, 470Ω1.2, C10.1, C11.2, C12.2, C15.2, C16.2, C17.2, C18.1, C8.2, C9.2
- net at Amplifier.12 (HPVDD): now also C17.1
- net at Amplifier.14 (VDD): now also DAC.1 (CPVDD), DAC.8 (AVDD), C10.2, C11.1, C18.2, C8.1, C9.1, FB1.2
- net at Amplifier.2 (INL+): now also C16.1
- net at Amplifier.3 (INR+): now also C15.1
- net at DAC.18 (LDOO): now also C5.1, C6.1
- net at DAC.2 (CAPP): now also C7.1
- net at DAC.4 (CAPM): now also C7.2
- net at DAC.5 (VNEG): now also C12.1
- net at DAC.6 (OUTL): now also 470Ω.1
- net at DAC.7 (OUTR): now also 470Ω1.1
Other:
- moved on the sheet: Amplifier, DAC, J1
