File: _autosave-esp-test.kicad_sch (KiCad schematic)
At the start: 44 parts, among them J1 AudioPlug3, U1 ESP32-S3-WROOM-1, U2 AP2112K-3.3

Commit message: work
Parts:
- added C21: 0.1 µF, symbol Device:C_Small
- added J2: Micro_SD_Card_Det1, symbol Connector:Micro_SD_Card_Det1
- added SW1: Volume Up, symbol Switch:SW_Push
- added SW2: Volume Down, symbol Switch:SW_Push
- 5.1 kΩ1: renamed from 5.1 kΩ
- 5.1 kΩ2: renamed from 5.1 kΩ
- JST PH 2.0 2-pin1: renamed from JST PH 2.0 2-pin
- USB-C Connector1: renamed from USB-C Connector
- renumbered 10kΩ to 10kΩ1, 10kΩ to 10kΩ2, 2kΩ to 2kΩ1, 4.7Ω to 4.7Ω1, 4.7Ω to 4.7Ω2, 470Ω to 470Ω1, 470Ω to 470Ω2, 470Ω to 470Ω3, Amplifier to Amplifier1, DAC to DAC1, PowerSwitch to PowerSwitch1
Connections:
- net GND: now also J2.6 (VSS), SW1.1, SW2.1
- net GNDA: now also C21.2, J2.10 (SHIELD)
- net at C4.2, FB1.1, U1.2 (3V3)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: now also C21.1, J2.4 (VDD)
- net at U1.20 (IO12): now also J2.7 (DAT0)
- net at U1.21 (IO13): now also J2.3 (CMD)
- net at U1.22 (IO14): now also J2.5 (CLK)
- net at U1.31 (IO38): now also J2.9 (DET)
- net at U1.8 (IO15): now also SW2.2
- net at U1.9 (IO16): now also SW1.2
- no-connect marks 3 -> 6
